Commit message: push before destructive tests

File: install/iir_base/share/iir_base/urdf/iirbot.urdf.xacro (robot description, xacro)
@@ -2,13 +2,13 @@
 <!-- Basic differential drive mobile base -->
 <robot xmlns:xacro="http://www.ros.org/wiki/xacro" name="iirbot">
-  <xacro:arg name="prefix" default="_" />
+  <xacro:arg name="prefix" default="" />
   <xacro:arg name="use_mock_hardware" default="false" />
-  <xacro:include filename="$(find iir_base)/src/urdf/iir_description.urdf.xacro" />
+  <xacro:include filename="$(find iir_base)/urdf/iir_description.urdf.xacro" />
   <!-- Import Rviz colors -->
-  <xacro:include filename="$(find iir_base)/src/urdf/iir.materials.xacro" />
+  <xacro:include filename="$(find iir_base)/urdf/iir.materials.xacro" />
   <!-- Import diffbot ros2_control description -->
-  <xacro:include filename="$(find iir_base)/src/urdf/iirbot.ros2_control.xacro" />
+  <xacro:include filename="$(find iir_base)/urdf/iirbot.ros2_control.xacro" />
   <xacro:iirbot_desc prefix="$(arg prefix)" />
   <xacro:iirbot_ros2_control
-    name="iirbot" prefix="$(arg prefix)" use_mock_hardware="$(arg use_mock_hardware)"/>
+    name="IirBot" prefix="$(arg prefix)" use_mock_hardware="$(arg use_mock_hardware)"/>
 </robot>

File: src/IIR_base/src/urdf/iir_description.urdf.xacro (robot description, xacro)
@@ -9,10 +9,10 @@
   <xacro:property name="base_height" value="0.17" />
   <xacro:property name="wheel_mass" value="0.3" /> <!-- arbitrary value for wheel mass -->
-  <xacro:property name="wheel_len" value="0.020" />
+  <xacro:property name="wheel_len" value="0.040" />
   <!-- wheels are .5m apart -->
   <xacro:property name="wheel_radius" value="0.05" />
   <xacro:property name="caster_wheel_mass" value="0.1" /> <!-- arbitrary value for caster wheel mass -->
   <xacro:property name="caster_wheel_radius" value="0.015" />
-  <xacro:property name="z_offset" value="-${base_height/2}" /> <!-- Space btw top of beam and the each joint -->
+  <xacro:property name="z_offset" value="-${base_height/3}" /> <!-- Space btw top of beam and the each joint -->
   <!-- Base Link -->
   <link name="${prefix}base_link">
@@ -42,5 +42,5 @@
       <parent link="${prefix}base_link"/>
       <child link="${prefix}left_wheel"/>
-      <origin xyz="0 -.45 ${z_offset}" rpy="0 0 0"/>
+      <origin xyz=".26 -.29 ${z_offset}" rpy="0 0 0"/>
       <axis xyz="0 1 0"/>
       <dynamics damping="0.2"/>
@@ -74,5 +74,5 @@
       <parent link="${prefix}base_link"/>
       <child link="${prefix}right_wheel"/>
-      <origin xyz="0 .45 ${z_offset}" rpy="0 0 0"/>
+      <origin xyz=".26 .29 ${z_offset}" rpy="0 0 0"/>
       <axis xyz="0 1 0"/>
       <dynamics damping="0.2"/>

File: src/IIR_base/src/urdf/iirbot.urdf.xacro (robot description, xacro)
@@ -2,5 +2,5 @@
 <!-- Basic differential drive mobile base -->
 <robot xmlns:xacro="http://www.ros.org/wiki/xacro" name="iirbot">
-  <xacro:arg name="prefix" default="_" />
+  <xacro:arg name="prefix" default="" />
   <xacro:arg name="use_mock_hardware" default="false" />
   <xacro:include filename="$(find iir_base)/urdf/iir_description.urdf.xacro" />
