Commit message: This package is mostly done, but needs cleaning

File: install/iir_base/share/iir_base/urdf/iir_description.urdf.xacro (robot description, xacro)
@@ -13,10 +13,10 @@
   <xacro:property name="wheel_radius" value="0.05" />
   <xacro:property name="caster_wheel_mass" value="0.1" /> <!-- arbitrary value for caster wheel mass -->
-  <xacro:property name="caster_wheel_radius" value="0.015" />
+  <xacro:property name="caster_wheel_radius" value="0.042" />
   <xacro:property name="z_offset" value="-${base_height/3}" /> <!-- Space btw top of beam and the each joint -->
   <!-- Base Link -->
-  <link name="${prefix}base_link">
+  <link name="base_link">
     <collision>
-      <origin xyz="0 0 0" rpy="0 0 0"/>
+      <origin xyz="0 0 ${base_height/2}" rpy="0 0 0"/>
       <geometry>
         <box size="${base_width} ${base_length} ${base_height}"/>
@@ -39,14 +39,16 @@
       </inertial>
     </link>
-    <joint name="${prefix}left_wheel_joint" type="continuous">
-      <parent link="${prefix}base_link"/>
-      <child link="${prefix}left_wheel"/>
-      <origin xyz=".26 -.29 ${z_offset}" rpy="0 0 0"/>
+  <gazebo reference="base_link">
+  </gazebo>
+    <joint name="left_wheel_joint" type="continuous">
+      <parent link="base_link"/>
+      <child link="left_wheel"/>
+      <origin xyz=".08 .29 ${z_offset}" rpy="0 0 0"/>
       <axis xyz="0 1 0"/>
       <dynamics damping="0.2"/>
-      <limit effort="100" velocity="1.0"/>
+      <limit effort="100" velocity="10.0"/>
     </joint>
     <!-- left wheel Link -->
-    <link name="${prefix}left_wheel">
+    <link name="left_wheel">
       <collision>
         <origin xyz="0 0 0" rpy="${PI/2} 0 0"/>
@@ -71,14 +73,24 @@
         </inertial>
       </link>
-    <joint name="${prefix}right_wheel_joint" type="continuous">
-      <parent link="${prefix}base_link"/>
-      <child link="${prefix}right_wheel"/>
-      <origin xyz=".26 .29 ${z_offset}" rpy="0 0 0"/>
+    <gazebo reference="left_wheel">
+      <mu1>1.0</mu1>
+      <mu2>1.0</mu2>
+      <kp>1000000.0</kp>
+      <kd>1.0</kd>
+      <minDepth>0.0001</minDepth>
+      <maxVel>10.0</maxVel>
+      <fdir1 value="0 1 0"/>
+      <material>Gazebo/DarkGrey</material>
+    </gazebo>
+    <joint name="right_wheel_joint" type="continuous">
+      <parent link="base_link"/>
+      <child link="right_wheel"/>
+      <origin xyz=".08 -.29 ${z_offset}" rpy="0 0 0"/>
       <axis xyz="0 1 0"/>
       <dynamics damping="0.2"/>
-      <limit effort="100" velocity="1.0"/>
+      <limit effort="100" velocity="10.0"/>
     </joint>
     <!-- right wheel Link -->
-    <link name="${prefix}right_wheel">
+    <link name="right_wheel">
       <collision>
         <origin xyz="0 0 0" rpy="${PI/2} 0 0"/>
@@ -103,11 +115,21 @@
         </inertial>
       </link>
-    <joint name="${prefix}caster_frontal_wheel_joint" type="fixed">
-      <parent link="${prefix}base_link"/>
-      <child link="${prefix}caster_frontal_wheel"/>
-      <origin xyz="${base_width/2 - caster_wheel_radius} 0 ${z_offset}" rpy="0 0 0"/>
+    <gazebo reference="right_wheel">
+      <mu1>1.0</mu1>
+      <mu2>1.0</mu2>
+      <kp>1000000.0</kp>
+      <kd>1.0</kd>
+      <minDepth>0.0001</minDepth>
+      <maxVel>10.0</maxVel>
+      <fdir1 value="0 1 0"/>
+      <material>Gazebo/DarkGrey</material>
+    </gazebo>
+    <!-- <joint name="caster_frontal_wheel_joint" type="fixed">
+      <parent link="base_link"/>
+      <child link="caster_frontal_wheel"/>
+      <origin xyz="${-base_width/2 - caster_wheel_radius} .29 ${z_offset}" rpy="0 0 0"/>
     </joint>
-    <!-- caster frontal wheel Link -->
-    <link name="${prefix}caster_frontal_wheel">
+     caster frontal wheel Link
+    <link name="caster_frontal_wheel">
       <collision>
         <origin xyz="0 0 0" rpy="0 0 0"/>
@@ -132,11 +154,12 @@
         </inertial>
       </link>
-    <joint name="${prefix}caster_rear_wheel_joint" type="fixed">
-      <parent link="${prefix}base_link"/>
-      <child link="${prefix}caster_rear_wheel"/>
-      <origin xyz="${-base_width/2 + caster_wheel_radius} 0 ${z_offset}" rpy="0 0 0"/>
+      -->
+    <joint name="caster_rear_wheel_joint" type="fixed">
+      <parent link="base_link"/>
+      <child link="caster_rear_wheel"/>
+      <origin xyz="-${base_width/2 + caster_wheel_radius} 0 ${z_offset}" rpy="0 0 0"/>
     </joint>
     <!-- caster rear wheel Link -->
-    <link name="${prefix}caster_rear_wheel">
+    <link name="caster_rear_wheel">
       <collision>
         <origin xyz="0 0 0" rpy="0 0 0"/>

File: install/iir_base/share/iir_base/urdf/iirbot.ros2_control.xacro (robot description, xacro)
@@ -4,22 +4,22 @@
     <ros2_control name="${name}" type="system">
       <xacro:unless value="${use_mock_hardware}">
-        <hardware>
-          <plugin>diff_drive_controller/DiffDriveController</plugin>
-          <param name="example_param_hw_start_duration_sec">0</param>
-          <param name="example_param_hw_stop_duration_sec">3.0</param>
-        </hardware>
+ <hardware>
+    <plugin>gz_ros2_control/GazeboSimSystem</plugin>
+              <param name="calculate_dynamics">true</param>
+<!-- having calculate dynamics o -->
+  </hardware>
       </xacro:unless>
       <xacro:if value="${use_mock_hardware}">
         <hardware>
           <plugin>mock_components/GenericSystem</plugin>
-          <param name="calculate_dynamics">true</param>
-        </hardware>
+  <param name="calculate_dynamics">true</param>
+          </hardware>
       </xacro:if>
-      <joint name="${prefix}left_wheel_joint">
+      <joint name="left_wheel_joint">
         <command_interface name="velocity"/>
         <state_interface name="position"/>
         <state_interface name="velocity"/>
       </joint>
-      <joint name="${prefix}right_wheel_joint">
+      <joint name="right_wheel_joint">
         <command_interface name="velocity"/>
         <state_interface name="position"/>
@@ -30,5 +30,29 @@
   <plugin filename="libgz_ros2_control-system.so" name="gz_ros2_control::GazeboSimROS2ControlPlugin">
     <parameters>$(find iir_base)/config/diffbot_controllers.yaml</parameters>
+  <controller_manager_prefix_node_name>controller_manager</controller_manager_prefix_node_name>
   </plugin>
+  <plugin filename="gz-sim-diff-drive-system" name="gz::sim::systems::DiffDrive">
+  <!-- Remove <ros> tag. -->
+  <!-- wheels -->
+  <left_joint>left_wheel_joint</left_joint>
+  <right_joint>right_wheel_joint</right_joint>
+  <!-- kinematics -->
+  <wheel_separation>0.58</wheel_separation>
+  <wheel_radius>0.05</wheel_radius> <!-- computed from <wheel_diameter> in the original plugin-->
+  <!-- limits -->
+  <max_linear_acceleration>100</max_linear_acceleration> <!-- computed from <max_linear_acceleration> in the original plugin-->
+  <topic>cmd_vel</topic> <!-- from <commant_topic> -->
+  <odom_topic>odom</odom_topic> <!-- from <odometry_topic> -->
+  <frame_id>odom</frame_id> <!-- from <odometry_frame> -->
+  <child_frame_id>base_link</child_frame_id> <!-- from <robot_base_frame> -->
+  <odom_publisher_frequency>30</odom_publisher_frequency> <!-- from <update_rate>-->
+  <tf_topic>/tf</tf_topic> <!-- Short topic name for tf output -->
+</plugin>
+<!-- <plugin filename="gz-sim-joint-state-publisher-system"
+  name="gz::sim::systems::JointStatePublisher">
+  <topic>joint_states</topic>
+  <joint_name>left_wheel_joint</joint_name>
+  <joint_name>right_wheel_joint</joint_name>
+</plugin> -->
 </gazebo>
   </xacro:macro>
